File: pcbgolf/board/pcbgolf-stock-4L.kicad_pcb (KiCad board)
At the start: 2 copper layers, 48.2 x 51 mm, 245 parts, among them J1 DCBARRELSMT, J2 MICRO_SD-0472192001, J3 USB-C-FEMALE, J4 CAN, J5 USB-C-FEMALEGCT, J6 USB-C-FEMALEGCT, J7 USB-C-FEMALEGCT, J8 USB-C-FEMALEGCT, Q1 SIS427-VI, Q2 NFET-DUAL-COMMON-SOURCE-QS5K2, Q3 NFET-DUAL-COMMON-SOURCE-QS5K2, Q4 NFET-DUAL-COMMON-SOURCE-QS5K2, Q5 NFET-DUAL-COMMON-SOURCE-QS5K2, Q6 NFET-DUAL-COMMON-SOURCE-QS5K2, Q7 NFET-DUAL-COMMON-SOURCE-QS5K2, Q8 NFET-DUAL-COMMON-SOURCE-QS5K2, Q9 NFET-DUAL-COMMON-SOURCE-QS5K2, SW1 SPST-2-4PIN, U1 AP62300T, U10 NCS20071XV, U11 NCS20071XV, U12 NCS20071XV, U13 TPS25942, U14 TPS25942, U15 TPS25942, U16 TPS25942, U2 AP62300T, U3 STM32H725ZGTx, U4 USB2517, U5 MCP2542FDT-E/MNY, U6 MCP2542FDT-E/MNY, U7 MCP2542FDT-E/MNY, U8 MCP2542FDT-E/MNY, U9 NCS20071XV, Y1 25MHz, Y2 24MHz

Commit message: Sync pcbgolf: measured part heights, 3D assembly bounding box, final board
Mirrors lblommesteyn/pcbgolf. The substantive change is that part heights are
now measured from the footprints' own STEP models rather than estimated: the
barrel jack is 11.00 mm, not the 9.00 mm assumed, so Z is 14.35 mm and every
previously reported volume was understated by about 5,300 mm^3.

Also adds bbox3d.py (the real PCBA bounding box, which is what the challenge
scores), step_assembly.py (a STEP built from that same geometry), and the
final LQFP-100 board with R11 not fitted, since the LQFP-100 package has no
PDR_ON pin for it to strap.

Co-Authored-By: Claude Opus 5 <noreply@anthropic.com>
Claude-Session: https://claude.ai/code/session_013nBHDXVrXKghy52w5PgN3h
Other:
- copper layers 2 -> 4
Changed lines of the file:
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@@
 	(layers
 		(0 "F.Cu" signal)
-		(2 "B.Cu" signal)
-		(4 "F.Adhes" user "F.Adhesive")
-		(6 "B.Adhes" user "B.Adhesive")
-		(8 "F.Paste" user)
-		(10 "B.Paste" user)
-		(12 "F.SilkS" user "F.Silkscreen")
-		(14 "B.SilkS" user "B.Silkscreen")
-		(16 "F.Mask" user)
-		(18 "B.Mask" user)
-		(20 "Dwgs.User" user "User.Drawings")
-		(22 "Cmts.User" user "User.Comments")
-		(24 "Eco1.User" user "User.Eco1")
-		(26 "Eco2.User" user "User.Eco2")
-		(28 "Edge.Cuts" user)
-		(30 "Margin" user)
-		(32 "F.CrtYd" user "F.Courtyard")
-		(34 "B.CrtYd" user "B.Courtyard")
-		(36 "F.Fab" user)
-		(38 "B.Fab" user)
+		(2 "In1.Cu" signal)
+		(4 "In2.Cu" signal)
+		(6 "B.Cu" signal)
+		(8 "F.Adhes" user "F.Adhesive")
+		(10 "B.Adhes" user "B.Adhesive")
+		(12 "F.Paste" user)
+		(14 "B.Paste" user)
+		(16 "F.SilkS" user "F.Silkscreen")
+		(18 "B.SilkS" user "B.Silkscreen")
+		(20 "F.Mask" user)
+		(22 "B.Mask" user)
+		(24 "Dwgs.User" user "User.Drawings")
+		(26 "Cmts.User" user "User.Comments")
+		(28 "Eco1.User" user "User.Eco1")
+		(30 "Eco2.User" user "User.Eco2")
+		(32 "Edge.Cuts" user)
+		(34 "Margin" user)
+		(36 "F.CrtYd" user "F.Courtyard")
+		(38 "B.CrtYd" user "B.Courtyard")
+		(40 "F.Fab" user)
+		(42 "B.Fab" user)
 	)
 	(setup
